Commit message: Replace RGB camera with RGB-D camera sensor

File: my_robot/urdf/my_robot.xacro (robot description, xacro)
@@ -160,4 +160,12 @@
   </joint>
   <!-- RGB CAMERA descriptor End-->
+  <!-- Add RGB-D camera -->
+  <joint name="camera_optical_joint" type="fixed">
+    <origin xyz="0 0 0" rpy="-1.5707 0 -1.5707"/>
+    <parent link="camera"/>
+    <child link="camera_link_optical"/>
+  </joint>
+  <link name="camera_link_optical">
+  </link>
   <!-- LASER descriptor start-->
   <link name="hokuyo">

Commit message: laser and camera link update

File: my_robot/urdf/my_robot.xacro (robot description, xacro)
@@ -160,5 +160,5 @@
   </joint>
   <!-- RGB CAMERA descriptor End-->
-  <!-- Add RGB-D camera -->
+  <link name="camera_link_optical"> </link>
   <joint name="camera_optical_joint" type="fixed">
     <origin xyz="0 0 0" rpy="-1.5707 0 -1.5707"/>
@@ -166,6 +166,4 @@
     <child link="camera_link_optical"/>
   </joint>
-  <link name="camera_link_optical">
-  </link>
   <!-- LASER descriptor start-->
   <link name="hokuyo">
